File: temperature_sensor.kicad_sch (KiCad schematic)
At the start: 29 parts, among them SW1 500SSP3S1M2QEA, U1 MMBT3904LT1G, U3 XIAO-SAMD21-SMD, U5 TMP37FT9Z

Commit message: sent for prod v1.0
Other:
- moved on the sheet: R4
Changed lines of the file:
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@@
 	(wire
 		(pts
-			(xy 57.15 273.05) (xy 57.15 271.78)
+			(xy 57.15 276.86) (xy 57.15 271.78)
 		)
 		(stroke
@@
 	(wire
 		(pts
-			(xy 49.53 273.05) (xy 57.15 273.05)
+			(xy 46.99 276.86) (xy 57.15 276.86)
 		)
 		(stroke
@@
 	(wire
 		(pts
-			(xy 46.99 252.73) (xy 49.53 252.73)
-		)
-		(stroke
-			(width 0)
-			(type default)
-		)
-	)
-	(wire
-		(pts
 			(xy 57.15 252.73) (xy 58.42 252.73)
 		)
@@
 	(wire
 		(pts
-			(xy 46.99 110.49) (xy 46.99 252.73)
+			(xy 46.99 110.49) (xy 46.99 256.54)
 		)
 		(stroke
@@
 	(symbol
 		(lib_id "CRGP2512F820R:CRGP2512F820R")
-		(at 49.53 262.89 270)
+		(at 46.99 266.7 270)
 		(unit 1)
 		(exclude_from_sim no)
@@
 		(fields_autoplaced yes)
 		(property "Reference" "R4"
-			(at 53.34 261.6199 90)
+			(at 50.8 265.4299 90)
 			(effects
 				(font
@@
 		)
 		(property "Value" "820"
-			(at 53.34 264.1599 90)
+			(at 50.8 267.9699 90)
 			(effects
 				(font
@@
 		)
 		(property "Footprint" "1_my_custom_library:RESC6332X65N"
-			(at 49.53 262.89 0)
+			(at 46.99 266.7 0)
 			(effects
 				(font
@@
 		)
 		(property "Datasheet" "~"
-			(at 49.53 262.89 0)
+			(at 46.99 266.7 0)
 			(effects
 				(font
@@
 		)
 		(property "Description" "Resistor"
-			(at 49.53 262.89 0)
-			(effects
-				(font
+			(at 46.99 266.7 0)
+			(effects
+				(font
